File: untitled.brd (EAGLE design)
At the start: 26 x 26 mm, 11 parts, among them IC1 NE555N

Commit message: Replaced fan JST with smaller pitch to match existing fan JST
Parts:
- FAN: value 2.54B-ZR -> B4B-ZR; device con-jst-custom:B4B-ZR2.5 -> con-jst-custom:B4B-ZR
Routing:
- net PWM: track 6.86 -> 7.50 mm
Changed lines of the file:
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@@
 <wire x1="26.0225" y1="26.025" x2="0" y2="26.025" width="0" layer="20"/>
 <wire x1="0" y1="26.025" x2="0" y2="0" width="0" layer="20"/>
-<text x="7.62" y="15.875" size="1.4224" layer="25">12V</text>
-<text x="6.35" y="9.8425" size="1.4224" layer="25">12V</text>
-<text x="7.62" y="13.6525" size="1.4224" layer="25">GND</text>
-<text x="7.3025" y="0.635" size="1.4224" layer="25">GND</text>
-<text x="7.62" y="20.0025" size="1.4224" layer="25">PWM</text>
+<text x="6.6675" y="16.51" size="1.4224" layer="25">12V</text>
+<text x="8.89" y="5.715" size="1.4224" layer="25" rot="R90">12V</text>
+<text x="6.6675" y="14.9225" size="1.4224" layer="25">GND</text>
+<text x="7.62" y="5.08" size="1.4224" layer="25" rot="R270">GND</text>
+<text x="6.6675" y="20.0025" size="1.4224" layer="25">PWM</text>
 </plain>
 <attributes>
@@
 <attribute name="VALUE" x="24.003" y="20.193" size="1.27" layer="28" rot="MR270"/>
 </element>
-<element name="FAN" library="con-jst-custom" package="B4B-ZR2.5" value="2.54B-ZR" x="4.445" y="17.78" smashed="yes" rot="R270">
-<attribute name="NAME" x="8.9775" y="21.9675" size="1.27" layer="25" rot="R90"/>
+<element name="FAN" library="con-jst-custom" package="B4B-ZR" package3d_urn="urn:adsk.eagle:package:7642/1" value="B4B-ZR" x="4.445" y="17.78" smashed="yes" rot="R270">
+<attribute name="MF" value="FARNELL" x="4.445" y="17.78" size="1.778" layer="27" rot="R270" display="off"/>
+<attribute name="MPN" value="B4B-ZR(LF)(SN)" x="4.445" y="17.78" size="1.778" layer="27" rot="R270" display="off"/>
+<attribute name="NAME" x="2.2825" y="21.82" size="1.27" layer="25"/>
+<attribute name="OC_FARNELL" value="1830916" x="4.445" y="17.78" size="1.778" layer="27" rot="R270" display="off"/>
+<attribute name="OC_NEWARK" value="37K9960" x="4.445" y="17.78" size="1.778" layer="27" rot="R270" display="off"/>
 <attribute name="VALUE" x="-1.595" y="22.8" size="1.27" layer="27" rot="R270"/>
 </element>
@@
 </element>
 <element name="SUPPLY" library="con-jst-custom" package="B2B-ZR2.5" value="2.52B-ZR" x="4.445" y="5.715" smashed="yes" rot="R270">
-<attribute name="NAME" x="7.5325" y="9.1475" size="1.27" layer="25" rot="R270"/>
+<attribute name="NAME" x="1.0125" y="10.0725" size="1.27" layer="25"/>
 <attribute name="VALUE" x="-1.595" y="8.195" size="1.27" layer="27" rot="R270"/>
 </element>
@@
 <via x="23.1775" y="4.1275" extent="1-16" drill="0.45" diameter="1.778"/>
 <via x="22.5425" y="7.3025" extent="1-16" drill="0.45" diameter="1.778"/>
+<wire x1="4.445" y1="15.53" x2="10.1727" y2="19.939" width="0" layer="19" extent="16-16"/>
+<wire x1="10.16" y1="12.3825" x2="4.445" y2="15.53" width="0" layer="19" extent="1-1"/>
+<wire x1="4.445" y1="4.4584" x2="10.16" y2="12.3825" width="0" layer="19" extent="1-1"/>
+<wire x1="22.5425" y1="7.3025" x2="10.16" y2="12.3825" width="0" layer="19" extent="1-1"/>
+<wire x1="23.1775" y1="4.1275" x2="22.5425" y2="7.3025" width="0" layer="19" extent="1-1"/>
 </signal>
 <signal name="Q">
@@
 <contactref element="FAN" pad="1"/>
 <contactref element="Q1" pad="1"/>
-<wire x1="11.1379" y1="21.971" x2="4.7879" y2="21.971" width="0.3048" layer="16"/>
-<wire x1="4.445" y1="21.6048" x2="4.445" y2="21.6281" width="0.3048" layer="16"/>
-<wire x1="4.7879" y1="21.971" x2="4.445" y2="21.6281" width="0.3048" layer="16"/>
+<wire x1="11.1379" y1="21.971" x2="6.3754" y2="21.971" width="0.3048" layer="16"/>
+<wire x1="6.3754" y1="21.971" x2="4.445" y2="20.0406" width="0.3048" layer="16"/>
+<wire x1="4.445" y1="20.03" x2="4.445" y2="20.0406" width="0.3048" layer="16"/>
 </signal>
 <signal name="CV">
@@
 <contactref element="R1" pad="2"/>
 <contactref element="SUPPLY" pad="1"/>
-<wire x1="4.445" y1="16.5234" x2="4.4316" y2="16.51" width="0.3048" layer="16"/>
-<wire x1="4.4316" y1="16.51" x2="3.175" y2="16.51" width="0.3048" layer="16"/>
-<wire x1="3.175" y1="16.51" x2="1.905" y2="15.24" width="0.3048" layer="16"/>
+<wire x1="4.445" y1="17.03" x2="4.33" y2="17.145" width="0.3048" layer="16"/>
+<wire x1="4.33" y1="17.145" x2="3.81" y2="17.145" width="0.3048" layer="16"/>
+<wire x1="3.81" y1="17.145" x2="1.905" y2="15.24" width="0.3048" layer="16"/>
 <wire x1="1.905" y1="9.5398" x2="4.445" y2="6.9998" width="0.3048" layer="16"/>
 <wire x1="1.905" y1="15.24" x2="1.905" y2="9.5398" width="0.3048" layer="16"/>
