File: untitled.sch (EAGLE design)
At the start: 11 parts, among them IC1 NE555N

Commit message: Replaced fan JST with smaller pitch to match existing fan JST
Parts:
- FAN: value 2.54B-ZR -> B4B-ZR; device con-jst-custom:2.54B-ZR -> con-jst-custom:B4B-ZR
Changed lines of the file:
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@@
 <part name="P+3" library="supply1" library_urn="urn:adsk.eagle:library:371" deviceset="+12V" device=""/>
 <part name="SUPPLY" library="con-jst-custom" deviceset="?2B-ZR" device="2.5"/>
-<part name="FAN" library="con-jst-custom" deviceset="?4B-ZR" device="2.5"/>
+<part name="FAN" library="con-jst-custom" deviceset="?4B-ZR" device="B" package3d_urn="urn:adsk.eagle:package:7642/1" value="B4B-ZR"/>
 <part name="Q1" library="zetex" library_urn="urn:adsk.eagle:library:418" deviceset="NMOSSOT23" device="" package3d_urn="urn:adsk.eagle:package:30981/1"/>
 <part name="GND5" library="supply1" library_urn="urn:adsk.eagle:library:371" deviceset="GND" device=""/>
